Commit message: Done

File: body.urdf (robot description, URDF)
Before this commit: robot robot, 3 links, 2 joints
Links:
- removed link FrontLet
- added link FrontLeg, mass 1; collision box size=1 1 1; visual box size=1 1 1
Joints:
- joint Torso_Front: child FrontLet -> FrontLeg

Commit message: Done

File: body.urdf (robot description, URDF)
Before this commit: robot robot, 3 links, 2 joints
Joints:
- joint Torso_Back: origin xyz=0 1 1 rpy=0 0 0 -> xyz=1 0 1 rpy=0 0 0
- joint Torso_Front: origin xyz=0 -1 1 rpy=0 0 0 -> xyz=2 0 1 rpy=0 0 0

Commit message: Done

File: body.urdf (robot description, URDF)
Before this commit: robot robot, 3 links, 2 joints
Links:
- added link BackLowerLeg, mass 1; collision box size=0.2 0.2 1; visual box size=0.2 0.2 1
- added link FrontLowerLeg, mass 1; collision box size=0.2 0.2 1; visual box size=0.2 0.2 1
- added link LeftLeg, mass 1; collision box size=1 0.2 0.2; visual box size=1 0.2 0.2
- added link LeftLowerLeg, mass 1; collision box size=0.2 0.2 1; visual box size=0.2 0.2 1
- added link RightLeg, mass 1; collision box size=1 0.2 0.2; visual box size=1 0.2 0.2
- added link RightLowerLeg, mass 1; collision box size=0.2 0.2 1; visual box size=0.2 0.2 1
- link BackLeg: geometry collision box size=0.2 1 0.2; visual box size=0.2 1 0.2
- link FrontLeg: geometry collision box size=0.2 1 0.2; visual box size=0.2 1 0.2
Joints:
- added joint BackLeg_BackLowerLeg: type revolute, parent BackLeg, child BackLowerLeg, origin xyz=0 -1 0 rpy=0 0 0, axis 1 0 0, limit lower=-3.14159 upper=3.14159 effort=0.0 velocity=0.0
- added joint FrontLeg_FrontLowerLeg: type revolute, parent FrontLeg, child FrontLowerLeg, origin xyz=0 1 0 rpy=0 0 0, axis 1 0 0, limit lower=-3.14159 upper=3.14159 effort=0.0 velocity=0.0
- added joint LeftLeg_LeftLowerLeg: type revolute, parent LeftLeg, child LeftLowerLeg, origin xyz=1 0 0 rpy=0 0 0, axis 1 0 0, limit lower=-3.14159 upper=3.14159 effort=0.0 velocity=0.0
- added joint RightLeg_RightLowerLeg: type revolute, parent RightLeg, child RightLowerLeg, origin xyz=-1 0 0 rpy=0 0 0, axis 1 0 0, limit lower=-3.14159 upper=3.14159 effort=0.0 velocity=0.0
- added joint Torso_Left: type revolute, parent Torso, child LeftLeg, origin xyz=0.5 0 1 rpy=0 0 0, axis 0 1 0, limit lower=-3.14159 upper=3.14159 effort=0.0 velocity=0.0
- added joint Torso_Right: type revolute, parent Torso, child RightLeg, origin xyz=-0.5 0 1 rpy=0 0 0, axis 0 1 0, limit lower=-3.14159 upper=3.14159 effort=0.0 velocity=0.0
- joint Torso_Back: axis 0 1 0 -> 1 0 0; origin xyz=1 0 1 rpy=0 0 0 -> xyz=0 -0.5 1 rpy=0 0 0
- joint Torso_Front: axis 0 1 0 -> 1 0 0; origin xyz=2 0 1 rpy=0 0 0 -> xyz=0 0.5 1 rpy=0 0 0

Commit message: Done

File: body.urdf (robot description, URDF)
Before this commit: robot robot, 9 links, 8 joints
Links:
- removed link BackLowerLeg
- removed link FrontLeg
- removed link FrontLowerLeg
- removed link LeftLeg
- removed link LeftLowerLeg
- removed link RightLeg
- removed link RightLowerLeg
- added link Back2, mass 1; collision box size=0.2 1 0.2; visual box size=0.2 1 0.2
Joints:
- removed joint BackLeg_BackLowerLeg
- removed joint FrontLeg_FrontLowerLeg
- removed joint LeftLeg_LeftLowerLeg
- removed joint RightLeg_RightLowerLeg
- removed joint Torso_Front
- removed joint Torso_Left
- removed joint Torso_Right
- added joint Back_Back2: type revolute, parent BackLeg, child Back2, origin xyz=0 -0.5 0.0 rpy=0 0 0, axis 0 1 0, limit lower=-3.14159 upper=3.14159 effort=0.0 velocity=0.0
- joint Torso_Back: axis 1 0 0 -> 0 0 1; origin xyz=0 -0.5 1 rpy=0 0 0 -> xyz=0 -1 0.5 rpy=0 0 0

Commit message: Done

File: body.urdf (robot description, URDF)
Before this commit: robot robot, 3 links, 2 joints
Links:
- removed link BackLeg
- added link Back, mass 1; collision box size=0.2 1 0.2; visual box size=0.2 1 0.2
- added link Back10, mass 1; collision box size=0.1 1 0.1; visual box size=0.1 1 0.1
- added link Back3, mass 1; collision box size=0.2 1 0.4; visual box size=0.2 1 0.4
- added link Back4, mass 1; collision box size=0.1 1 0.1; visual box size=0.1 1 0.1
- added link Back5, mass 1; collision box size=0.4 1 0.2; visual box size=0.4 1 0.2
- added link Back6, mass 1; collision box size=0.2 1 0.4; visual box size=0.2 1 0.4
- added link Back7, mass 1; collision box size=0.1 1 0.1; visual box size=0.1 1 0.1
- added link Back8, mass 1; collision box size=0.4 1 0.2; visual box size=0.4 1 0.2
- added link Back9, mass 1; collision box size=0.2 1 0.4; visual box size=0.2 1 0.4
- link Torso: geometry collision box size=0.3 0.3 0.3; visual box size=0.3 0.3 0.3
Joints:
- added joint Back2_Back3: type revolute, parent Back2, child Back3, origin xyz=0 -1 0.0 rpy=0 0 0, axis 0 0 1, limit lower=-3.14159 upper=3.14159 effort=0.0 velocity=0.0
- added joint Back3_Back4: type revolute, parent Back3, child Back4, origin xyz=0 -1 0.0 rpy=0 0 0, axis 0 0 1, limit lower=-3.14159 upper=3.14159 effort=0.0 velocity=0.0
- added joint Back4_Back5: type revolute, parent Back4, child Back5, origin xyz=0 -1 0.0 rpy=0 0 0, axis 1 0 0, limit lower=-3.14159 upper=3.14159 effort=0.0 velocity=0.0
- added joint Back5_Back6: type revolute, parent Back5, child Back6, origin xyz=0 -1 0.0 rpy=0 0 0, axis 0 0 1, limit lower=-3.14159 upper=3.14159 effort=0.0 velocity=0.0
- added joint Back6_Back7: type revolute, parent Back6, child Back7, origin xyz=0 -1 0.0 rpy=0 0 0, axis 0 0 1, limit lower=-3.14159 upper=3.14159 effort=0.0 velocity=0.0
- added joint Back7_Back8: type revolute, parent Back7, child Back8, origin xyz=0 -1 0.0 rpy=0 0 0, axis 1 0 0, limit lower=-3.14159 upper=3.14159 effort=0.0 velocity=0.0
- added joint Back8_Back9: type revolute, parent Back8, child Back9, origin xyz=0 -1 0.0 rpy=0 0 0, axis 0 0 1, limit lower=-3.14159 upper=3.14159 effort=0.0 velocity=0.0
- added joint Back9_Back10: type revolute, parent Back9, child Back10, origin xyz=0 -1 0.0 rpy=0 0 0, axis 0 0 1, limit lower=-3.14159 upper=3.14159 effort=0.0 velocity=0.0
- joint Back_Back2: axis 0 1 0 -> 0 1 1; parent BackLeg -> Back
- joint Torso_Back: axis 0 0 1 -> 1 0 1; child BackLeg -> Back; origin xyz=0 -1 0.5 rpy=0 0 0 -> xyz=0.0 -0.3 0.15 rpy=0 0 0

Commit message: Done

File: body.urdf (robot description, URDF)
Before this commit: robot robot, 11 links, 10 joints
Links:
- removed link Back
- removed link Back10
- removed link Torso
- added link Back0, mass 1; collision box size=0.34889728844377343 0.5524828620342417 0.31873923668167986; visual box size=0.34889728844377343 0.5524828620342417 0.31873923668167986
- added link Back1, mass 1; collision box size=0.44229336420901527 0.16253920165012575 0.21924634137232002; visual box size=0.44229336420901527 0.16253920165012575 0.21924634137232002
- link Back2: geometry collision box size=0.33445181344268826 0.24907946636810574 0.6248506489317329; visual box size=0.33445181344268826 0.24907946636810574 0.6248506489317329
- link Back3: geometry collision box size=0.19745104306769787 0.381996555932692 0.2931745755569982; visual box size=0.19745104306769787 0.381996555932692 0.2931745755569982
- link Back4: geometry collision box size=0.42304675443486583 0.06029837785878441 0.16118381356109995; visual box size=0.42304675443486583 0.06029837785878441 0.16118381356109995
- link Back5: geometry collision box size=0.2106812514628546 0.2275441116106331 0.5049405678269879; visual box size=0.2106812514628546 0.2275441116106331 0.5049405678269879
- link Back6: geometry collision box size=0.4066438002398369 0.46876882545773124 0.2753514505822974; visual box size=0.4066438002398369 0.46876882545773124 0.2753514505822974
- link Back7: geometry collision box size=0.17646319881730987 0.5102352024747743 0.46918916204958727; visual box size=0.17646319881730987 0.5102352024747743 0.46918916204958727
- link Back8: geometry collision box size=0.6156704003584799 0.624477072091163 0.3477944892744054; visual box size=0.6156704003584799 0.624477072091163 0.3477944892744054
- link Back9: geometry collision box size=0.3287813940604739 0.17778513822874847 0.3250072802012345; visual box size=0.3287813940604739 0.17778513822874847 0.3250072802012345
Joints:
- removed joint Back9_Back10
- removed joint Back_Back2
- removed joint Torso_Back
- added joint Back0_Back1: type revolute, parent Back0, child Back1, origin xyz=0 -0.27624143101712084 0.0 rpy=0 0 0, axis 0 0 1, limit lower=-3.14159 upper=3.14159 effort=0.0 velocity=0.0
- added joint Back1_Back2: type revolute, parent Back1, child Back2, origin xyz=0 -0.16253920165012575 0.0 rpy=0 0 0, axis 0 0 1, limit lower=-3.14159 upper=3.14159 effort=0.0 velocity=0.0
- joint Back2_Back3: axis 0 0 1 -> 1 0 0; origin xyz=0 -1 0.0 rpy=0 0 0 -> xyz=0 -0.24907946636810574 0.0 rpy=0 0 0
- joint Back3_Back4: origin xyz=0 -1 0.0 rpy=0 0 0 -> xyz=0 -0.381996555932692 0.0 rpy=0 0 0
- joint Back4_Back5: axis 1 0 0 -> 0 0 1; origin xyz=0 -1 0.0 rpy=0 0 0 -> xyz=0 -0.06029837785878441 0.0 rpy=0 0 0
- joint Back5_Back6: axis 0 0 1 -> 1 0 0; origin xyz=0 -1 0.0 rpy=0 0 0 -> xyz=0 -0.2275441116106331 0.0 rpy=0 0 0
- joint Back6_Back7: origin xyz=0 -1 0.0 rpy=0 0 0 -> xyz=0 -0.46876882545773124 0.0 rpy=0 0 0
- joint Back7_Back8: axis 1 0 0 -> 0 0 1; origin xyz=0 -1 0.0 rpy=0 0 0 -> xyz=0 -0.5102352024747743 0.0 rpy=0 0 0
- joint Back8_Back9: axis 0 0 1 -> 1 0 0; origin xyz=0 -1 0.0 rpy=0 0 0 -> xyz=0 -0.624477072091163 0.0 rpy=0 0 0

Commit message: Done

File: body.urdf (robot description, URDF)
Before this commit: robot robot, 10 links, 9 joints
Links:
- link Back0: geometry collision box size=0.35310646610102026 0.5694636006708913 0.10261864644962179; visual box size=0.35310646610102026 0.5694636006708913 0.10261864644962179
- link Back1: geometry collision box size=0.3076893861794662 0.6296818036837586 0.08253798782140517; visual box size=0.3076893861794662 0.6296818036837586 0.08253798782140517
- link Back2: geometry collision box size=0.3066392257073435 0.5887593817517427 0.17148042592285168; visual box size=0.3066392257073435 0.5887593817517427 0.17148042592285168
- link Back3: geometry collision box size=0.25551479857521187 0.41856813945054117 0.5955588269361973; visual box size=0.25551479857521187 0.41856813945054117 0.5955588269361973
- link Back4: geometry collision box size=0.43196865901504966 0.4205103251321404 0.16331382283876417; visual box size=0.43196865901504966 0.4205103251321404 0.16331382283876417
- link Back5: geometry collision box size=0.08075396385941108 0.5213562883829796 0.5374836080381042; visual box size=0.08075396385941108 0.5213562883829796 0.5374836080381042
- link Back6: geometry collision box size=0.3699129134347183 0.568706725989157 0.16333216001166606; visual box size=0.3699129134347183 0.568706725989157 0.16333216001166606
- link Back7: geometry collision box size=0.5258489468567287 0.3418316774320898 0.5699421200886392; visual box size=0.5258489468567287 0.3418316774320898 0.5699421200886392
- link Back8: geometry collision box size=0.30153767416509275 0.5889962117312335 0.15128400426722846; visual box size=0.30153767416509275 0.5889962117312335 0.15128400426722846
- link Back9: geometry collision box size=0.22361440540322805 0.3117002636000902 0.2831656783337718; visual box size=0.22361440540322805 0.3117002636000902 0.2831656783337718
Joints:
- joint Back0_Back1: origin xyz=0 -0.27624143101712084 0.0 rpy=0 0 0 -> xyz=0 -0.28473180033544565 0.0 rpy=0 0 0
- joint Back1_Back2: origin xyz=0 -0.16253920165012575 0.0 rpy=0 0 0 -> xyz=0 -0.6296818036837586 0.0 rpy=0 0 0
- joint Back2_Back3: origin xyz=0 -0.24907946636810574 0.0 rpy=0 0 0 -> xyz=0 -0.5887593817517427 0.0 rpy=0 0 0
- joint Back3_Back4: origin xyz=0 -0.381996555932692 0.0 rpy=0 0 0 -> xyz=0 -0.41856813945054117 0.0 rpy=0 0 0
- joint Back4_Back5: origin xyz=0 -0.06029837785878441 0.0 rpy=0 0 0 -> xyz=0 -0.4205103251321404 0.0 rpy=0 0 0
- joint Back5_Back6: origin xyz=0 -0.2275441116106331 0.0 rpy=0 0 0 -> xyz=0 -0.5213562883829796 0.0 rpy=0 0 0
- joint Back6_Back7: origin xyz=0 -0.46876882545773124 0.0 rpy=0 0 0 -> xyz=0 -0.568706725989157 0.0 rpy=0 0 0
- joint Back7_Back8: origin xyz=0 -0.5102352024747743 0.0 rpy=0 0 0 -> xyz=0 -0.3418316774320898 0.0 rpy=0 0 0
- joint Back8_Back9: origin xyz=0 -0.624477072091163 0.0 rpy=0 0 0 -> xyz=0 -0.5889962117312335 0.0 rpy=0 0 0

Commit message: Done

File: body.urdf (robot description, URDF)
Before this commit: robot robot, 10 links, 9 joints
Links:
- link Back0: geometry collision box size=0.5859167134605248 0.13398518386646724 0.6302379595996388; visual box size=0.5859167134605248 0.13398518386646724 0.6302379595996388
- link Back1: geometry collision box size=0.08203967803553541 0.34331192862626025 0.4022155237464073; visual box size=0.08203967803553541 0.34331192862626025 0.4022155237464073
- link Back2: geometry collision box size=0.2392717188268411 0.3434712795897565 0.51098605502738; visual box size=0.2392717188268411 0.3434712795897565 0.51098605502738
- link Back3: geometry collision box size=0.25568286290897013 0.25522318329839977 0.23463952198423724; visual box size=0.25568286290897013 0.25522318329839977 0.23463952198423724
- link Back4: geometry collision box size=0.5459538366417771 0.3030642524184837 0.5501197764250361; visual box size=0.5459538366417771 0.3030642524184837 0.5501197764250361
- link Back5: geometry collision box size=0.40191102800540096 0.20896699341141742 0.2942599389429492; visual box size=0.40191102800540096 0.20896699341141742 0.2942599389429492
- link Back6: geometry collision box size=0.5552562244839012 0.3683232430614659 0.6166375536563524; visual box size=0.5552562244839012 0.3683232430614659 0.6166375536563524
- link Back7: geometry collision box size=0.2572243761119811 0.09928425556790446 0.47933400375609614; visual box size=0.2572243761119811 0.09928425556790446 0.47933400375609614
- link Back8: geometry collision box size=0.5151881089222463 0.10999196025331914 0.1365381081819554; visual box size=0.5151881089222463 0.10999196025331914 0.1365381081819554
- link Back9: geometry collision box size=0.2931416957532884 0.5351898892401323 0.5702453791261204; visual box size=0.2931416957532884 0.5351898892401323 0.5702453791261204
Joints:
- joint Back0_Back1: origin xyz=0 -0.28473180033544565 0.0 rpy=0 0 0 -> xyz=0 -0.06699259193323362 0.0 rpy=0 0 0
- joint Back1_Back2: origin xyz=0 -0.6296818036837586 0.0 rpy=0 0 0 -> xyz=0 -0.34331192862626025 0.0 rpy=0 0 0
- joint Back2_Back3: origin xyz=0 -0.5887593817517427 0.0 rpy=0 0 0 -> xyz=0 -0.3434712795897565 0.0 rpy=0 0 0
- joint Back3_Back4: origin xyz=0 -0.41856813945054117 0.0 rpy=0 0 0 -> xyz=0 -0.25522318329839977 0.0 rpy=0 0 0
- joint Back4_Back5: origin xyz=0 -0.4205103251321404 0.0 rpy=0 0 0 -> xyz=0 -0.3030642524184837 0.0 rpy=0 0 0
- joint Back5_Back6: origin xyz=0 -0.5213562883829796 0.0 rpy=0 0 0 -> xyz=0 -0.20896699341141742 0.0 rpy=0 0 0
- joint Back6_Back7: origin xyz=0 -0.568706725989157 0.0 rpy=0 0 0 -> xyz=0 -0.3683232430614659 0.0 rpy=0 0 0
- joint Back7_Back8: origin xyz=0 -0.3418316774320898 0.0 rpy=0 0 0 -> xyz=0 -0.09928425556790446 0.0 rpy=0 0 0
- joint Back8_Back9: origin xyz=0 -0.5889962117312335 0.0 rpy=0 0 0 -> xyz=0 -0.10999196025331914 0.0 rpy=0 0 0

File: summerbod.urdf (robot description, URDF)
Before this commit: robot robot, 2 links, 1 joints
Links:
- added link 1, mass 1; collision box size=0.23141977527356736 0.40221436352356643 0.5290213944703528; visual box size=0.23141977527356736 0.40221436352356643 0.5290213944703528
- added link 2, mass 1; collision box size=0.5685629896046613 0.4513942133539595 0.3560583796156521; visual box size=0.5685629896046613 0.4513942133539595 0.3560583796156521
- added link 3, mass 1; collision box size=0.6187727642303491 0.38490950728437556 0.5738796890120152; visual box size=0.6187727642303491 0.38490950728437556 0.5738796890120152
- added link 4, mass 1; collision box size=0.23526613899081564 0.5407112008768975 0.07524567265590146; visual box size=0.23526613899081564 0.5407112008768975 0.07524567265590146
- added link 5, mass 1; collision box size=0.260488638358942 0.1753916310861672 0.5466291255262725; visual box size=0.260488638358942 0.1753916310861672 0.5466291255262725
- added link 7, mass 1; collision box size=0.2917187113022627 0.09451742137517813 0.2744010633366496; visual box size=0.2917187113022627 0.09451742137517813 0.2744010633366496
- added link 8, mass 1; collision box size=0.40100196431116725 0.27219102340033496 0.06244015784054996; visual box size=0.40100196431116725 0.27219102340033496 0.06244015784054996
- added link 9, mass 1; collision box size=0.421734015279684 0.1008034360929153 0.2357177506137289; visual box size=0.421734015279684 0.1008034360929153 0.2357177506137289
- link 0: geometry collision box size=0.09144791958810611 0.20585598888906406 0.6173457215742961; visual box size=0.09144791958810611 0.20585598888906406 0.6173457215742961
- link 6: geometry collision box size=0.16804938141647088 0.35953962674212675 0.10431613137192183; visual box size=0.16804938141647088 0.35953962674212675 0.10431613137192183
Joints:
- added joint Joint0_1: type revolute, parent 0, child 1, origin xyz=0.0 0.10292799444453203 0.0 rpy=0 0 0, axis 0 0 1, limit lower=-3.14159 upper=3.14159 effort=0.0 velocity=0.0
- added joint Joint0_2: type revolute, parent 0, child 2, origin xyz=0.0 0.0 -0.30867286078714806 rpy=0 0 0, axis 0 0 1, limit lower=-3.14159 upper=3.14159 effort=0.0 velocity=0.0
- added joint Joint0_4: type revolute, parent 0, child 4, origin xyz=0.0 -0.10292799444453203 0.0 rpy=0 0 0, axis 0 0 1, limit lower=-3.14159 upper=3.14159 effort=0.0 velocity=0.0
- added joint Joint0_7: type revolute, parent 0, child 7, origin xyz=-0.045723959794053054 0.0 0.0 rpy=0 0 0, axis 0 0 1, limit lower=-3.14159 upper=3.14159 effort=0.0 velocity=0.0
- added joint Joint0_9: type revolute, parent 0, child 9, origin xyz=0.045723959794053054 0.0 0.0 rpy=0 0 0, axis 0 0 1, limit lower=-3.14159 upper=3.14159 effort=0.0 velocity=0.0
- added joint Joint1_5: type revolute, parent 1, child 5, origin xyz=0.11570988763678368 0.20110718176178322 0.0 rpy=0 0 0, axis 0 0 1, limit lower=-3.14159 upper=3.14159 effort=0.0 velocity=0.0
- added joint Joint2_3: type revolute, parent 2, child 3, origin xyz=0.0 0.0 -0.3560583796156521 rpy=0 0 0, axis 0 0 1, limit lower=-3.14159 upper=3.14159 effort=0.0 velocity=0.0
- added joint Joint3_8: type revolute, parent 3, child 8, origin xyz=0.30938638211517455 0.0 -0.2869398445060076 rpy=0 0 0, axis 0 0 1, limit lower=-3.14159 upper=3.14159 effort=0.0 velocity=0.0
- joint Joint0_6: origin xyz=-1 0 0.0 rpy=0 0 0 -> xyz=0.0 0.0 0.30867286078714806 rpy=0 0 0
