Commit message: Its half working

File: summerbod.urdf (robot description, URDF)
Before this commit: robot robot, 10 links, 9 joints
Links:
- removed link 5
- removed link 6
- removed link 7
- removed link 8
- removed link 9
- link 0: geometry collision box size=0.6364888641375821 0.2673231155287903 0.12426664436457398; visual box size=0.6364888641375821 0.2673231155287903 0.12426664436457398
- link 1: geometry collision box size=0.12641850069504357 0.06058086531835977 0.1548204443912568; visual box size=0.12641850069504357 0.06058086531835977 0.1548204443912568
- link 2: geometry collision box size=0.28633451992328096 0.3117070361049873 0.07226050965242498; visual box size=0.28633451992328096 0.3117070361049873 0.07226050965242498
- link 3: geometry collision box size=0.2104837372075032 0.45951438652512483 0.42073120124667385; visual box size=0.2104837372075032 0.45951438652512483 0.42073120124667385
- link 4: geometry collision box size=0.09806985839475874 0.19543693086149871 0.45345300711021763; visual box size=0.09806985839475874 0.19543693086149871 0.45345300711021763
Joints:
- removed joint Joint0_1
- removed joint Joint0_2
- removed joint Joint0_4
- removed joint Joint0_6
- removed joint Joint0_7
- removed joint Joint0_9
- removed joint Joint1_5
- removed joint Joint2_3
- removed joint Joint3_8
- added joint Joint_One_0_1: type revolute, parent 0, child 1, origin xyz=0.31824443206879105 0.0 0.0 rpy=0 0 0, axis 0 0 1, limit lower=-3.14159 upper=3.14159 effort=0.0 velocity=0.0
- added joint Joint_One_0_2: type revolute, parent 0, child 2, origin xyz=-0.31824443206879105 0.0 0.0 rpy=0 0 0, axis 0 0 1, limit lower=-3.14159 upper=3.14159 effort=0.0 velocity=0.0
- added joint Joint_One_1_4: type revolute, parent 1, child 4, origin xyz=0.06320925034752178 0.0 0.0774102221956284 rpy=0 0 0, axis 0 1 0, limit lower=-3.14159 upper=3.14159 effort=0.0 velocity=0.0
- added joint Joint_One_2_3: type revolute, parent 2, child 3, origin xyz=-0.14316725996164048 0.0 0.03613025482621249 rpy=0 0 0, axis 0 1 0, limit lower=-3.14159 upper=3.14159 effort=0.0 velocity=0.0
- added joint Joint_Two_0_1: type revolute, parent 0, child 1, origin xyz=0.31824443206879105 0.0 0.0 rpy=0 0 0, axis 0 1 0, limit lower=-3.14159 upper=3.14159 effort=0.0 velocity=0.0
- added joint Joint_Two_0_2: type revolute, parent 0, child 2, origin xyz=-0.31824443206879105 0.0 0.0 rpy=0 0 0, axis 0 1 0, limit lower=-3.14159 upper=3.14159 effort=0.0 velocity=0.0
- added joint Joint_Two_1_4: type revolute, parent 1, child 4, origin xyz=0.06320925034752178 0.0 0.0774102221956284 rpy=0 0 0, axis 1 0 0, limit lower=-3.14159 upper=3.14159 effort=0.0 velocity=0.0
- added joint Joint_Two_2_3: type revolute, parent 2, child 3, origin xyz=-0.14316725996164048 0.0 0.03613025482621249 rpy=0 0 0, axis 1 0 0, limit lower=-3.14159 upper=3.14159 effort=0.0 velocity=0.0
