Commit message: DONE

File: bodyCubes1.urdf (robot description, URDF)
Before this commit: robot robot, 5 links, 4 joints
Links:
- added link 10, mass 1; collision box size=0.5262600927051058 0.3187326147792265 0.27511222920572337; visual box size=0.5262600927051058 0.3187326147792265 0.27511222920572337
- added link 11, mass 1; collision box size=0.29877216096138803 0.18433918405024974 0.08526085673439718; visual box size=0.29877216096138803 0.18433918405024974 0.08526085673439718
- added link 12, mass 1; collision box size=0.1478126938848034 0.17878202613476535 0.2868191785885785; visual box size=0.1478126938848034 0.17878202613476535 0.2868191785885785
- added link 13, mass 1; collision box size=0.08437921598754056 0.06917108398183608 0.5663728114154447; visual box size=0.08437921598754056 0.06917108398183608 0.5663728114154447
- added link 14, mass 1; collision box size=0.5364870947827844 0.37079901497593387 0.4200853710943426; visual box size=0.5364870947827844 0.37079901497593387 0.4200853710943426
- added link 5, mass 1; collision box size=0.25556634267594625 0.5626421046267103 0.08991419796219104; visual box size=0.25556634267594625 0.5626421046267103 0.08991419796219104
- added link 6, mass 1; collision box size=0.14005233252152943 0.3725193170485193 0.4504699428898423; visual box size=0.14005233252152943 0.3725193170485193 0.4504699428898423
- added link 7, mass 1; collision box size=0.48741459150974503 0.6016260903715984 0.44408471987593445; visual box size=0.48741459150974503 0.6016260903715984 0.44408471987593445
- added link 8, mass 1; collision box size=0.18470646221449483 0.4122753028170861 0.06533824922944728; visual box size=0.18470646221449483 0.4122753028170861 0.06533824922944728
- added link 9, mass 1; collision box size=0.5436710973436856 0.6548998494694167 0.11215306460485461; visual box size=0.5436710973436856 0.6548998494694167 0.11215306460485461
- link 0: geometry collision box size=0.5147726417641815 0.31234294849850697 0.5666531109150288; visual box size=0.5147726417641815 0.31234294849850697 0.5666531109150288
- link 1: geometry collision box size=0.343285629271628 0.12042072484101948 0.3205031012722702; visual box size=0.343285629271628 0.12042072484101948 0.3205031012722702
- link 2: geometry collision box size=0.10145114909033931 0.4672343755853351 0.1381346703027354; visual box size=0.10145114909033931 0.4672343755853351 0.1381346703027354
- link 3: geometry collision box size=0.3288811959861877 0.4862099856529685 0.4642651201850984; visual box size=0.3288811959861877 0.4862099856529685 0.4642651201850984
- link 4: geometry collision box size=0.604823914295755 0.422386432687125 0.060041497724690196; visual box size=0.604823914295755 0.422386432687125 0.060041497724690196
Joints:
- removed joint Joint0_2
- removed joint Joint1_3
- removed joint Joint2_4
- added joint Joint10_14: type revolute, parent 10, child 14, origin xyz=0.5262600927051058 0.0 0.0 rpy=0 0 0, axis 1 0 0, limit lower=-3.14159 upper=3.14159 effort=0.0 velocity=0.0
- added joint Joint1_2: type revolute, parent 1, child 2, origin xyz=-0.171642814635814 0.0 0.1602515506361351 rpy=0 0 0, axis 1 0 0, limit lower=-3.14159 upper=3.14159 effort=0.0 velocity=0.0
- added joint Joint2_13: type revolute, parent 2, child 13, origin xyz=-0.050725574545169655 0.0 0.0690673351513677 rpy=0 0 0, axis 0 1 0, limit lower=-3.14159 upper=3.14159 effort=0.0 velocity=0.0
- added joint Joint2_3: type revolute, parent 2, child 3, origin xyz=-0.050725574545169655 -0.23361718779266755 0.0 rpy=0 0 0, axis 0 1 0, limit lower=-3.14159 upper=3.14159 effort=0.0 velocity=0.0
- added joint Joint2_6: type revolute, parent 2, child 6, origin xyz=-0.050725574545169655 0.23361718779266755 0.0 rpy=0 0 0, axis 0 1 0, limit lower=-3.14159 upper=3.14159 effort=0.0 velocity=0.0
- added joint Joint2_8: type revolute, parent 2, child 8, origin xyz=-0.10145114909033931 0.0 0.0 rpy=0 0 0, axis 1 0 0, limit lower=-3.14159 upper=3.14159 effort=0.0 velocity=0.0
- added joint Joint3_4: type revolute, parent 3, child 4, origin xyz=0.16444059799309385 -0.24310499282648426 0.0 rpy=0 0 0, axis 1 0 0, limit lower=-3.14159 upper=3.14159 effort=0.0 velocity=0.0
- added joint Joint3_5: type revolute, parent 3, child 5, origin xyz=0.0 -0.24310499282648426 0.2321325600925492 rpy=0 0 0, axis 0 1 0, limit lower=-3.14159 upper=3.14159 effort=0.0 velocity=0.0
- added joint Joint3_7: type revolute, parent 3, child 7, origin xyz=0.0 -0.4862099856529685 0.0 rpy=0 0 0, axis 0 1 0, limit lower=-3.14159 upper=3.14159 effort=0.0 velocity=0.0
- added joint Joint6_9: type revolute, parent 6, child 9, origin xyz=0.07002616626076472 0.18625965852425966 0.0 rpy=0 0 0, axis 1 0 0, limit lower=-3.14159 upper=3.14159 effort=0.0 velocity=0.0
- added joint Joint7_11: type revolute, parent 7, child 11, origin xyz=-0.24370729575487252 -0.3008130451857992 0.0 rpy=0 0 0, axis 1 0 0, limit lower=-3.14159 upper=3.14159 effort=0.0 velocity=0.0
- added joint Joint9_10: type revolute, parent 9, child 10, origin xyz=0.5436710973436856 0.0 0.0 rpy=0 0 0, axis 1 0 0, limit lower=-3.14159 upper=3.14159 effort=0.0 velocity=0.0
- added joint Joint9_12: type revolute, parent 9, child 12, origin xyz=0.2718355486718428 0.0 -0.056076532302427304 rpy=0 0 0, axis 0 1 0, limit lower=-3.14159 upper=3.14159 effort=0.0 velocity=0.0
- joint Joint0_1: origin xyz=-0.2828979428675391 0.0 0.0 rpy=0 0 0 -> xyz=0.0 0.0 0.2833265554575144 rpy=0 0 0
