Commit message: Done

File: bodyCubes35000.urdf (robot description, URDF)
Before this commit: robot robot, 15 links, 14 joints
Links:
- link 0: geometry collision box size=-0.019912867810943057 -0.003003152259968949 0.0101444509077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; visual box size=-0.019912867810943057 -0.003003152259968949 0.0101444509077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
- link 1: geometry collision box size=0.0036899268018527136 0.0038975605843356393 0.0086982283687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; visual box size=0.0036899268018527136 0.0038975605843356393 0.0086982283687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
- link 10: geometry collision box size=-0.002895241093151556 0.01234879211619785 -0.00601411685003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; visual box size=-0.002895241093151556 0.01234879211619785 -0.00601411685003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
- link 11: geometry collision box size=0.09843511811222852 0.6548613699167258 0.5162330867146326; visual box size=0.09843511811222852 0.6548613699167258 0.5162330867146326
- link 12: geometry collision box size=0.32809078106228484 0.5709458609418969 0.36268088475380256; visual box size=0.32809078106228484 0.5709458609418969 0.36268088475380256
- link 13: geometry collision box size=0.22069288347067992 0.5309458798801718 0.3581013117376408; visual box size=0.22069288347067992 0.5309458798801718 0.3581013117376408
- link 14: geometry collision box size=0.51915485301931 0.11766196884038324 0.07755067159729384; visual box size=0.51915485301931 0.11766196884038324 0.07755067159729384
- link 2: geometry collision box size=0.001953063035655686 0.0057276379713404576 -0.0005435034542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; visual box size=0.001953063035655686 0.0057276379713404576 -0.0005435034542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
- link 3: geometry collision box size=0.007748571737265832 0.00188624280504012 0.0052041855130467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; visual box size=0.007748571737265832 0.00188624280504012 0.0052041855130467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
- link 4: geometry collision box size=0.00012655313083713375 -8.247279417844452e-06 1.35708716844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; visual box size=0.00012655313083713375 -8.247279417844452e-06 1.35708716844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
- link 5: geometry collision box size=0.4213209850176221 0.49930763597848415 0.11594505860444462; visual box size=0.4213209850176221 0.49930763597848415 0.11594505860444462
- link 6: geometry collision box size=0.19847177514885259 0.6385373264531089 0.3518521306200392; visual box size=0.19847177514885259 0.6385373264531089 0.3518521306200392
- link 7: geometry collision box size=0.6583802798106129 0.08784304728938988 0.17277498260682012; visual box size=0.6583802798106129 0.08784304728938988 0.17277498260682012
- link 8: geometry collision box size=0.637578053376735 0.274687618767292 0.5608488477711255; visual box size=0.637578053376735 0.274687618767292 0.5608488477711255
- link 9: geometry collision box size=0.11004149540329067 0.10903264637241326 0.20662349608622796; visual box size=0.11004149540329067 0.10903264637241326 0.20662349608622796
Joints:
- removed joint Joint10_14
- removed joint Joint2_13
- removed joint Joint2_6
- removed joint Joint3_4
- removed joint Joint3_7
- removed joint Joint6_9
- removed joint Joint9_10
- removed joint Joint9_12
- added joint Joint1_4: type revolute, parent 1, child 4, origin xyz=0.0 -0.0019487802921678197 0.004349114184385349 rpy=0 0 0, axis 0 1 0, limit lower=-3.14159 upper=3.14159 effort=0.0 velocity=0.0
- added joint Joint3_13: type revolute, parent 3, child 13, origin xyz=0.0 0.00094312140252006 0.0026020927565233933 rpy=0 0 0, axis 0 1 0, limit lower=-3.14159 upper=3.14159 effort=0.0 velocity=0.0
- added joint Joint4_6: type revolute, parent 4, child 6, origin xyz=0.0 8.247279417844452e-06 0.0 rpy=0 0 0, axis 0 1 0, limit lower=-3.14159 upper=3.14159 effort=0.0 velocity=0.0
- added joint Joint4_7: type revolute, parent 4, child 7, origin xyz=-6.327656541856687e-05 4.123639708922226e-06 0.0 rpy=0 0 0, axis 1 0 0, limit lower=-3.14159 upper=3.14159 effort=0.0 velocity=0.0
- added joint Joint6_10: type revolute, parent 6, child 10, origin xyz=0.09923588757442629 -0.31926866322655445 0.0 rpy=0 0 0, axis 1 0 0, limit lower=-3.14159 upper=3.14159 effort=0.0 velocity=0.0
- added joint Joint8_12: type revolute, parent 8, child 12, origin xyz=0.637578053376735 0.0 0.0 rpy=0 0 0, axis 1 0 0, limit lower=-3.14159 upper=3.14159 effort=0.0 velocity=0.0
- added joint Joint8_14: type revolute, parent 8, child 14, origin xyz=0.3187890266883675 0.137343809383646 0.0 rpy=0 0 0, axis 0 1 0, limit lower=-3.14159 upper=3.14159 effort=0.0 velocity=0.0
- added joint Joint8_9: type revolute, parent 8, child 9, origin xyz=0.3187890266883675 -0.137343809383646 0.0 rpy=0 0 0, axis 0 1 0, limit lower=-3.14159 upper=3.14159 effort=0.0 velocity=0.0
- joint Joint0_1: origin xyz=0.0 0.0 0.2833265554575144 rpy=0 0 0 -> xyz=-0.0 -0.0 0.005072225453860074 rpy=0 0 0
- joint Joint1_2: origin xyz=-0.171642814635814 0.0 0.1602515506361351 rpy=0 0 0 -> xyz=0.0018449634009263568 0.0 0.004349114184385349 rpy=0 0 0
- joint Joint2_3: origin xyz=-0.050725574545169655 -0.23361718779266755 0.0 rpy=0 0 0 -> xyz=0.000976531517827843 0.0028638189856702288 -0.0 rpy=0 0 0
- joint Joint2_8: origin xyz=-0.10145114909033931 0.0 0.0 rpy=0 0 0 -> xyz=0.001953063035655686 0.0 -0.0 rpy=0 0 0
- joint Joint3_5: origin xyz=0.0 -0.24310499282648426 0.2321325600925492 rpy=0 0 0 -> xyz=0.0 0.00094312140252006 -0.0026020927565233933 rpy=0 0 0
- joint Joint7_11: axis 1 0 0 -> 0 1 0; origin xyz=-0.24370729575487252 -0.3008130451857992 0.0 rpy=0 0 0 -> xyz=-0.32919013990530643 0.04392152364469494 0.0 rpy=0 0 0
